File: kicad/flamingo.kicad_pcb (KiCad board)
At the start: 4 copper layers, 53.3 x 85.1 mm, 48 parts, among them J1 SWD, J2 Conn_01x02, J3 Conn_01x02, J4 Conn_01x03, J5 Conn_01x02, Q0 Q_PMOS_GSD, Q1 Q_PMOS_GSD, Q2 Q_PMOS_GSD, SW0 SW, SW1 SW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

Commit message: Revision 2
Changed the following items on the schematic and layout.
 - Disconnected SDO from U1 and U2
 - Changed U3 and U4 pull up resistors to have a source of 3.3V, not VCC
 - Added 1k I2C resistors
 - Fixed U5 BYPASS connection error
 - Updated schematic photo
Parts:
- added R200: 1k, Resistor_SMD:R_0603_1608Metric_Pad0.98x0.95mm_HandSolder, F.Cu at (133.6, 115.3)
- added R201: 1k, Resistor_SMD:R_0603_1608Metric_Pad0.98x0.95mm_HandSolder, F.Cu at (124.5, 110.2)
- moved C501 8.52 mm to (151.4, 98.0), turned to 0 degrees
- moved C502 3.14 mm to (145.3, 94.5)
- moved U5 1.52 mm to (149.2, 93.7)
- moved C500 1.05 mm to (149.4, 87.9), turned to 90 degrees
Connections:
- C501 pad 2: Net-(C501-Pad2) -> GND
- C502 pad 1: Net-(C501-Pad2) -> Net-(C502-Pad1)
- R300 pad 1: VCC -> +3V3
- R400 pad 1: VCC -> +3V3
- U1 pad 15: PB1_SDO -> Net-(U1-Pad15)
- U2 pad 2: PB1_SDO -> Net-(U2-Pad2)
- U5 pad 4: Net-(C501-Pad2) -> Net-(C502-Pad1)
Routing:
- net PB1_SDO: track 53.3 -> 0.00 mm, vias 2 -> 0
- net Net-(C501-Pad2): track 8.80 -> 0.00 mm
- net VCC: track 34.7 -> 27.8 mm, vias 10 -> 5
- net +3V3: track 53.6 -> 59.6 mm, vias 16 -> 18
- net Net-(C502-Pad1): track 0.00 -> 3.10 mm
- net PA15_I2C1_SCL: track 30.6 -> 33.1 mm
- net PB7_I2C1_SDA: track 29.4 -> 31.2 mm
- net GND: track 74.9 -> 75.7 mm, vias 45 -> 46
